File: MQTTbug.kicad_sch (KiCad schematic)
At the start: 23 parts, among them J1 Conn_01x02, J10 Conn_01x03, J11 Conn_01x04, J12 Conn_01x03, J2 Conn_01x02, J3 Conn_01x06, J4 Conn_01x04, J5 Conn_01x04, J6 Conn_01x04, J7 Conn_01x04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

Commit message: 2023-02-08: worked on PCB layout
Parts:
- J10, J12: footprint Connector_PinSocket_2.54mm:PinSocket_1x03_P2.54mm_Vertical -> Connector_PinHeader_2.54mm:PinHeader_1x03_P2.54mm_Vertical
Connections:
- net SW_PWR: now reaches J10.2 (Pin_2), J9.6 (Pin_6)
Changed lines of the file:
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@@
+    (effects (font (size 1.27 1.27)) (justify left bottom))
+  )
+  (label "SW_PWR" (at 175.26 153.67 0)
     (effects (font (size 1.27 1.27)) (justify left bottom))
   )
@@
     (property "Reference" "J12" (id 0) (at 229.87 144.8902 0))
     (property "Value" "Conn_01x03" (id 1) (at 229.87 147.4271 0))
-    (property "Footprint" "Connector_PinSocket_2.54mm:PinSocket_1x03_P2.54mm_Vertical" (id 2) (at 229.87 152.4 0)
+    (property "Footprint" "Connector_PinHeader_2.54mm:PinHeader_1x03_P2.54mm_Vertical" (id 2) (at 229.87 152.4 0)
       (effects (font (size 1.27 1.27)) hide)
     )
@@
       (effects (font (size 1.27 1.27)) (justify left))
     )
-    (property "Footprint" "Connector_PinSocket_2.54mm:PinSocket_1x03_P2.54mm_Vertical" (id 2) (at 196.85 153.67 0)
+    (property "Footprint" "Connector_PinHeader_2.54mm:PinHeader_1x03_P2.54mm_Vertical" (id 2) (at 196.85 153.67 0)
       (effects (font (size 1.27 1.27)) hide)
     )
@@
     )
     (path "/67a3e386-15db-4f94-9925-f50f444a5bd7"
-      (reference "J10") (unit 1) (value "Conn_01x03") (footprint "Connector_PinSocket_2.54mm:PinSocket_1x03_P2.54mm_Vertical")
+      (reference "J10") (unit 1) (value "Conn_01x03") (footprint "Connector_PinHeader_2.54mm:PinHeader_1x03_P2.54mm_Vertical")
     )
     (path "/2c7b32a0-5fd7-4db6-977a-150574e469ff"
@@
     )
     (path "/518b86e9-f59c-4f73-b19a-33521db7f705"
-      (reference "J12") (unit 1) (value "Conn_01x03") (footprint "Connector_PinSocket_2.54mm:PinSocket_1x03_P2.54mm_Vertical")
+      (reference "J12") (unit 1) (value "Conn_01x03") (footprint "Connector_PinHeader_2.54mm:PinHeader_1x03_P2.54mm_Vertical")
     )
     (path "/8e20d17c-3471-4547-9d6f-5b37d649f1fb"
